File: shiftled.kicad_pcb (KiCad board)
At the start: 2 copper layers, 24 parts, among them J1 Conn_01x07_Pin, U1 74HC595

Commit message: move capasitor
Parts:
- moved C1 6.80 mm to (90.5, 66.5)
Changed lines of the file:
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@@
 	(footprint "Capacitor_SMD:C_0805_2012Metric"
 		(layer "F.Cu")
-		(at 83.95 64.5)
+		(at 90.45 66.5)
 		(descr "Capacitor SMD 0805 (2012 Metric), square (rectangular) end terminal, IPC-7351 nominal, (Body size source: IPC-SM-782 page 76, https://www.pcb-3d.com/wordpress/wp-content/uploads/ipc-sm-782a_amendment_1_and_2.pdf, https://docs.google.com/spreadsheets/d/1BsfQQcO9C6DZCsRaXUlFlo91Tg2WpOkGARC1WS5S8t0/edit?usp=sharing), generated with kicad-footprint-generator")
 		(tags "capacitor")

Commit message: routing parts
Parts:
- moved R9 30.0 mm to (66.0, 84.0)
- moved R10 20.8 mm to (66.0, 91.0)
- moved R13 20.7 mm to (65.9, 87.5), turned to 180 degrees
- moved R11 20.5 mm to (75.0, 79.0), turned to 90 degrees
- moved R12 12.3 mm to (65.9, 81.0), turned to 180 degrees
- moved C1 6.58 mm to (91.5, 73.0), turned to 180 degrees
- moved R1 0.12 mm to (100.0, 67.5)
Routing:
- net +5V: track 0.00 -> 56.1 mm
- net Net-(J1-Pin_3): track 0.00 -> 39.4 mm, vias 0 -> 1
- net Net-(J1-Pin_4): track 0.00 -> 38.2 mm, vias 0 -> 1
- net Net-(J1-Pin_6): track 0.00 -> 33.2 mm
- net Net-(J1-Pin_5): track 0.00 -> 32.8 mm, vias 0 -> 1
- net GND: track 0.00 -> 25.9 mm, vias 0 -> 16
- net Net-(J1-Pin_2): track 0.00 -> 24.5 mm
- net Net-(U1-QB): track 0.00 -> 22.3 mm
- net Net-(U1-QH): track 0.00 -> 20.9 mm
- net Net-(U1-QC): track 0.00 -> 19.5 mm
- net Net-(U1-QG): track 0.00 -> 19.4 mm
- net Net-(U1-QF): track 0.00 -> 17.8 mm
- net Net-(U1-QD): track 0.00 -> 17.2 mm
- net Net-(U1-QA): track 0.00 -> 17.0 mm
- net Net-(U1-QE): track 0.00 -> 16.0 mm
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- added copper zone on B.Cu, net GND
Other:
- board outline added: 51 x 40.5 mm
